File: pi-gpio-mux.kicad_pcb (KiCad board)
At the start: 2 copper layers, 65 x 56 mm, 35 parts, among them J1 Raspberry_Pi_2_3, J2 Raw, J3 Buffered, J4 Register-1, J5 Register-2, J6 Clk1, J7 Clk2, U1 74AHCT245, U10 74AHCT574, U11 74AHCT574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

Commit message: Bus raw -> buffers
Routing:
- net Pin36-GPIO16: track 53.4 -> 58.9 mm
- net User3: track 37.9 -> 43.3 mm
- net Pin28-GPIO1: track 47.7 -> 52.9 mm
- net Pin38-GPIO20: track 49.9 -> 54.8 mm
- net User1: track 36.3 -> 40.8 mm
- net Pin31-GPIO6: track 47.1 -> 51.5 mm
- net User4: track 40.0 -> 44.3 mm, vias 2 -> 3
- net Pin33-GPIO13: track 48.6 -> 52.9 mm, vias 2 -> 3
- net Pin40-GPIO21: track 50.2 -> 54.5 mm
- net Pin29-GPIO5: track 45.5 -> 49.8 mm
- net Pin32-GPIO12: track 48.4 -> 51.9 mm, vias 2 -> 3
- net User2: track 37.7 -> 41.2 mm, vias 2 -> 3
- net Pin26-GPIO7: track 47.5 -> 50.8 mm, vias 2 -> 3
- net Pin35-GPIO19: track 45.5 -> 48.6 mm, vias 2 -> 3
- net Pin27-GPIO0: track 43.1 -> 45.8 mm, vias 2 -> 3
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
Commit message: Start power connections.
Routing:
- net VCC: track 141.5 -> 180.9 mm, vias 16 -> 12
- net GND: track 128.3 -> 155.2 mm, vias 0 -> 5
- net /CLK1: track 40.6 -> 53.0 mm
- net /CLK2: track 51.0 -> 62.7 mm, vias 6 -> 3
- net Pin16-GPIO23: track 48.0 -> 48.7 mm
- added copper zone on B.Cu, net GND
Other:
- net class Default: via_drill 0.5 -> 0.4
